File: GESC/GESC.kicad_pcb (KiCad board)
At the start: 4 copper layers, 140.5 x 80 mm, 73 parts, among them J1 gates_A, J2 gates_B, J3 SH2, J4 SH1, J5 gates_C, J6 SH3, Q1 TOLL, Q10 TOLL, Q11 TOLL, Q12 TOLL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

Commit message: asdf
Parts:
- added C20: 470nF, Capacitor_SMD:C_1210_3225Metric, F.Cu at (70.5, 116.7)
- added C24: 470nF, Capacitor_SMD:C_1210_3225Metric, F.Cu at (70.5, 131.4)
- added REF**: MountingHole_3.2mm_M3_ISO7380, MountingHole:MountingHole_3.2mm_M3_ISO7380, F.Cu at (187.5, 147.0)
- added REF**: MountingHole_3.2mm_M3_ISO7380, MountingHole:MountingHole_3.2mm_M3_ISO7380, F.Cu at (57.0, 77.0)
- added REF**: MountingHole_3.2mm_M3_ISO7380, MountingHole:MountingHole_3.2mm_M3_ISO7380, F.Cu at (187.5, 77.0)
- added REF**: MountingHole_3.2mm_M3_ISO7380, MountingHole:MountingHole_3.2mm_M3_ISO7380, F.Cu at (57.0, 147.0)
- J3, J4, J6: footprint Connector_PinHeader_2.00mm:PinHeader_2x01_P2.00mm_Vertical_SMD -> Connector_PinHeader_2.00mm:PinHeader_1x02_P2.00mm_Vertical_SMD_Pin1Right
- TH1: value 100k NTC -> 10k NTC
- moved C15 5.55 mm to (70.5, 92.0)
- moved C24 2.80 mm to (70.5, 128.2)
- moved C20 2.60 mm to (70.5, 113.4)
- moved C19 1.90 mm to (70.5, 110.1)
- moved C15 1.80 mm to (70.5, 95.3)
- moved C16 1.55 mm to (70.5, 98.5)
- moved C23 1.55 mm to (70.5, 125.0)
- moved C18 1.15 mm to (70.5, 106.8)
- moved C17 0.80 mm to (70.5, 101.8)
- moved C21 0.80 mm to (70.5, 121.7)
- turned J3 to 0 degrees
- turned J4 to 0 degrees
- turned J6 to 0 degrees
Routing:
- net Net-(J4-Pin_1): track 41.5 -> 11.2 mm
- net Net-(J6-Pin_2): track 41.9 -> 11.6 mm
- net Net-(J3-Pin_1): track 41.5 -> 11.4 mm
- net Net-(Q10-S-Pad2): track 43.3 -> 14.2 mm
- net Net-(Q14-S-Pad2): track 41.9 -> 13.7 mm
- net Net-(Q4-S-Pad2): track 41.2 -> 13.3 mm
- net GND: track 122.7 -> 142.8 mm
- net +BATT: track 27.3 -> 30.0 mm

Commit message: asdf
Parts:
- removed the C15 at (70.5, 92.0)
- removed the C15 at (70.5, 95.3)
- removed the C16 at (70.5, 98.5)
- removed the C18 at (70.5, 106.8)
- removed the C20 at (70.5, 113.4)
- removed the C20 at (70.5, 116.7)
- removed the C22 at (70.5, 137.0)
- removed the C23 at (70.5, 125.0)
- removed the C24 at (70.5, 128.2)
- removed the C24 at (70.5, 131.4)
- removed C25, C26, C27, C28: 330uF, lcsc:CAP-SMD_BD12.5-L13.5-W13.5-FD-1
- added ?: , , F.Cu at (166.4, 57.0)
- added ?: , , F.Cu at (38.1, 57.0)
- added ?: , , F.Cu at (158.4, 57.0)
- added ?: , , F.Cu at (46.1, 57.0)
- added C1: 470nF, Capacitor_SMD:C_1210_3225Metric, F.Cu at (170.0, 74.1)
- added C1: 470nF, Capacitor_SMD:C_1210_3225Metric, F.Cu at (34.6, 39.6)
- added C10: 470nF, Capacitor_SMD:C_1210_3225Metric, F.Cu at (170.0, 39.7)
- added C10: 470nF, Capacitor_SMD:C_1210_3225Metric, F.Cu at (34.6, 74.0)
- added C15: 470nF, Capacitor_SMD:C_1210_3225Metric, F.Cu at (34.6, 36.5)
- added C15: 470nF, Capacitor_SMD:C_1210_3225Metric, F.Cu at (170.0, 77.3)
- added C16: 470nF, Capacitor_SMD:C_1210_3225Metric, F.Cu at (34.6, 33.2)
- added C16: 470nF, Capacitor_SMD:C_1210_3225Metric, F.Cu at (170.0, 80.5)
- added C18: 470nF, Capacitor_SMD:C_1210_3225Metric, F.Cu at (170.0, 83.7)
- added C18: 470nF, Capacitor_SMD:C_1210_3225Metric, F.Cu at (34.6, 30.1)
- added C2: 470nF, Capacitor_SMD:C_1210_3225Metric, F.Cu at (170.0, 70.9)
- added C2: 470nF, Capacitor_SMD:C_1210_3225Metric, F.Cu at (34.6, 42.9)
- added C20: 470nF, Capacitor_SMD:C_1210_3225Metric, F.Cu at (170.0, 23.7)
- added C22: 470nF, Capacitor_SMD:C_1210_3225Metric, F.Cu at (170.0, 30.1)
- added C22: 470nF, Capacitor_SMD:C_1210_3225Metric, F.Cu at (34.6, 83.7)
- added C23: 470nF, Capacitor_SMD:C_1210_3225Metric, F.Cu at (34.6, 80.5)
- added C23: 470nF, Capacitor_SMD:C_1210_3225Metric, F.Cu at (170.0, 33.3)
- added C24: 470nF, Capacitor_SMD:C_1210_3225Metric, F.Cu at (170.0, 36.5)
- added C24: 470nF, Capacitor_SMD:C_1210_3225Metric, F.Cu at (34.6, 77.2)
- added C3: 470nF, Capacitor_SMD:C_1210_3225Metric, F.Cu at (34.6, 46.0)
- added C3: 470nF, Capacitor_SMD:C_1210_3225Metric, F.Cu at (170.0, 67.7)
- added C4: 470nF, Capacitor_SMD:C_1210_3225Metric, F.Cu at (170.0, 64.5)
- added C4: 470nF, Capacitor_SMD:C_1210_3225Metric, F.Cu at (34.6, 49.2)
- added C5: 470nF, Capacitor_SMD:C_1210_3225Metric, F.Cu at (170.0, 61.3)
- added C5: 470nF, Capacitor_SMD:C_1210_3225Metric, F.Cu at (34.6, 52.5)
- added C6: 470nF, Capacitor_SMD:C_1210_3225Metric, F.Cu at (34.6, 61.2)
- added C6: 470nF, Capacitor_SMD:C_1210_3225Metric, F.Cu at (170.0, 52.5)
- added C7: 470nF, Capacitor_SMD:C_1210_3225Metric, F.Cu at (170.0, 49.3)
- added C7: 470nF, Capacitor_SMD:C_1210_3225Metric, F.Cu at (34.6, 64.5)
- added C8: 470nF, Capacitor_SMD:C_1210_3225Metric, F.Cu at (34.6, 67.7)
- added C8: 470nF, Capacitor_SMD:C_1210_3225Metric, F.Cu at (170.0, 46.1)
- added C9: 470nF, Capacitor_SMD:C_1210_3225Metric, F.Cu at (170.0, 42.9)
- added C9: 470nF, Capacitor_SMD:C_1210_3225Metric, F.Cu at (34.6, 70.8)
- R12, R13, R16, R17, R52, R55, R58, R61, R9: value 0.5mR -> 0.2mR
- TH1: value 10k NTC -> 10k ntc
- moved C21 137.4 mm to (170.0, 26.9), turned to 0 degrees
- moved J5 119.2 mm to (84.0, 53.0)
- moved C19 93.6 mm to (34.6, 23.6)
- moved C17 83.1 mm to (34.6, 26.9)
- moved J1 70.7 mm to (152.5, 53.0)
- moved J6 67.3 mm to (152.5, 77.0)
- moved R18 66.5 mm to (153.8, 46.5)
- moved R47 66.1 mm to (153.6, 71.8), turned to 0 degrees
- moved R61 65.1 mm to (147.3, 77.2)
- moved R59 65.0 mm to (153.8, 44.4)
- moved R51 64.9 mm to (153.6, 66.6)
- moved R57 64.9 mm to (153.6, 68.1)
- moved R60 64.9 mm to (153.6, 69.6)
- moved R56 64.9 mm to (153.8, 43.0)
- moved Q17 64.9 mm to (146.7, 41.3)
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Connections:
- J1 pad 2: Net-(J1-Pin_2) -> Phase_C
- J1 pad 4: Phase_A -> Net-(J1-Pin_4)
- J5 pad 2: Phase_C -> Net-(J5-Pin_2)
- J5 pad 4: Net-(J5-Pin_4) -> Phase_A
- R1 pad 1: Net-(J1-Pin_2) -> Net-(J5-Pin_2)
- R12 pad 2: Net-(J3-Pin_1) (its old number) -> GND
- R13 pad 2: Net-(J4-Pin_1) (its old number) -> GND
- R16 pad 2: Net-(J4-Pin_1) (its old number) -> GND
- R17 pad 2: Net-(J3-Pin_1) (its old number) -> GND
- R18 pad 1: Net-(J5-Pin_4) -> Net-(J1-Pin_4)
- R2 pad 1: Net-(J1-Pin_3) -> Net-(J5-Pin_3)
- R3 pad 1: Net-(J1-Pin_2) -> Net-(J5-Pin_2)
- R4 pad 1: Net-(J1-Pin_3) -> Net-(J5-Pin_3)
- R47 pad 1: Net-(J5-Pin_3) -> Net-(J1-Pin_3)
- R48 pad 1: Net-(J5-Pin_4) -> Net-(J1-Pin_4)
- R49 pad 1: Net-(J1-Pin_2) -> Net-(J5-Pin_2)
- R50 pad 1: Net-(J1-Pin_3) -> Net-(J5-Pin_3)
- R51 pad 1: Net-(J5-Pin_3) -> Net-(J1-Pin_3)
- R52 pad 2: Net-(J6-Pin_2) -> GND
- R53 pad 1: Net-(J1-Pin_2) -> Net-(J5-Pin_2)
- R54 pad 1: Net-(J1-Pin_3) -> Net-(J5-Pin_3)
- R55 pad 2: Net-(J4-Pin_1) (its old number) -> GND
- R56 pad 1: Net-(J5-Pin_4) -> Net-(J1-Pin_4)
- R57 pad 1: Net-(J5-Pin_3) -> Net-(J1-Pin_3)
- R58 pad 2: Net-(J6-Pin_2) -> GND
- R59 pad 1: Net-(J5-Pin_4) -> Net-(J1-Pin_4)
- R60 pad 1: Net-(J5-Pin_3) -> Net-(J1-Pin_3)
- R61 pad 2: Net-(J6-Pin_2) -> GND
- R9 pad 2: Net-(J3-Pin_1) (its old number) -> GND
Routing:
- net GND: track 142.8 -> 265.2 mm
- net +BATT: track 30.0 -> 120.5 mm
- net Net-(J6-Pin_2): track 11.6 -> 0.00 mm
- net Net-(J3-Pin_1) (its old number): track 11.4 -> 0.00 mm
- net Net-(J4-Pin_1) (its old number): track 11.2 -> 0.00 mm
- net Net-(J5-Pin_4): track 11.0 -> 0.00 mm
- net Net-(J1-Pin_2): track 10.0 -> 0.00 mm
- net Net-(J1-Pin_4): track 0.00 -> 9.86 mm
- net Net-(J5-Pin_2): track 0.00 -> 9.76 mm
- net Phase_A: track 12.9 -> 18.3 mm
- net Net-(J6-Pin_1): track 13.7 -> 8.52 mm
- net Phase_B: track 12.5 -> 17.3 mm
- net Net-(J3-Pin_1): track 14.2 -> 10.8 mm
- net Net-(J4-Pin_1): track 13.3 -> 10.1 mm
- net Phase_C: track 8.01 -> 10.8 mm
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- added copper zone on F.Cu, net Net-(J3-Pin_1)
- added copper zone on F.Cu, net Net-(J4-Pin_1)
- added copper zone on F.Cu, net Net-(J6-Pin_1)
Other:
- board size 140.5 x 80 mm -> 140.5 x 90 mm

Commit message: asdf
Routing:
- net +BATT: track 120.5 -> 139.4 mm
